File: pcb/stm32f103cb_lcd32.sch (EAGLE design)
At the start: 75 parts, among them IC3 STM32F103C8, IC4 L1117-3.3, Q2 32768Hz, Q3 8MHz, Q5 MMBT2222

Commit message: Element values
Parts:
- Q1: value (none) -> MMBT2907
- R2: value 220 -> 1K
Changed lines of the file:
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@@
 <setting verticaltext="up"/>
 </settings>
-<grid distance="0.1" unitdist="inch" unit="inch" style="lines" multiple="1" display="yes" altdistance="0.01" altunitdist="inch" altunit="inch"/>
+<grid distance="0.1" unitdist="inch" unit="inch" style="lines" multiple="1" display="no" altdistance="0.01" altunitdist="inch" altunit="inch"/>
 <layers>
 <layer number="1" name="Top" color="4" fill="1" visible="no" active="no"/>
@@
 <part name="GND8" library="rs485" deviceset="GND" device=""/>
 <part name="LED1" library="led" deviceset="LED" device="CHIP-LED0805" value="Green"/>
-<part name="R2" library="rc-master-smd" deviceset="R_" device="0603" value="220"/>
+<part name="R2" library="rc-master-smd" deviceset="R_" device="0603" value="1K"/>
 <part name="SWD1" library="jtag" deviceset="SWD-6" device=""/>
 <part name="G1" library="battery" deviceset="1220SMT" device="" value="3V"/>
@@
 <part name="R4" library="rc-master-smd" deviceset="R_" device="0603" value="22"/>
 <part name="R5" library="rc-master-smd" deviceset="R_" device="0603" value="10K"/>
-<part name="Q1" library="semiconductor" deviceset="PNP-" device="SOT23"/>
+<part name="Q1" library="semiconductor" deviceset="PNP-" device="SOT23" value="MMBT2907"/>
 <part name="+3V33" library="supply1" deviceset="+3V3" device=""/>
 <part name="D1" library="semicon-smd-ipc" deviceset="D-" device="SMB"/>
